File: eagle/NOS01/NOS01.brd (EAGLE design)
At the start: 93.7 x 71.1 mm, 41 parts, among them IC1 TL072P, IC2 TL072P, T1 2SC1815, T2 2SC1815

Commit message: Update eagle files
Parts:
- R1: value 1k -> 10k
- turned C1 to 270 degrees
- turned C2 to 270 degrees
Other:
- board text added: "Use Pin Socket"
Changed lines of the file:
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@@
 <hole x="91.44" y="68.58" drill="3.2"/>
 <hole x="91.44" y="2.54" drill="3.2"/>
+<text x="19.05" y="55.88" size="1.27" layer="48">Use Pin Socket</text>
+<wire x1="31.75" y1="55.88" x2="17.78" y2="55.88" width="0" layer="48"/>
+<wire x1="17.78" y1="55.88" x2="15.24" y2="53.34" width="0" layer="48"/>
 </plain>
 <attributes>
@@
 </autorouter>
 <elements>
-<element name="C1" library="rcl" package="E2,5-6" value="47uF" x="68.58" y="31.75" rot="R90"/>
+<element name="C1" library="rcl" package="E2,5-6" value="47uF" x="68.58" y="31.75" rot="R270"/>
 <element name="C10" library="rcl" package="C025-024X044" value="0.1uF" x="44.45" y="40.64"/>
-<element name="C2" library="rcl" package="E2,5-6" value="47uF" x="68.58" y="39.37" rot="R90"/>
+<element name="C2" library="rcl" package="E2,5-6" value="47uF" x="68.58" y="39.37" rot="R270"/>
 <element name="C3" library="rcl" package="C050-045X075" value="1uF" x="25.4" y="48.26"/>
 <element name="C4" library="rcl" package="C050-045X075" value="1uF" x="20.32" y="27.94" rot="R90"/>
@@
 <element name="JP6" library="pinhead" package="1X02" value="BLUE" x="57.15" y="20.32"/>
 <element name="LED1" library="led" package="LED3MM" value="GREEN" x="71.12" y="46.99" rot="R270"/>
-<element name="R1" library="rcl" package="0207/7" value="1k" x="74.93" y="50.8"/>
+<element name="R1" library="rcl" package="0207/7" value="10k" x="74.93" y="50.8"/>
 <element name="R10" library="rcl" package="0207/7" value="10k" x="55.88" y="49.53" rot="R270"/>
 <element name="R11" library="rcl" package="0207/7" value="100k" x="60.96" y="44.45" rot="R270"/>
@@
 <contactref element="JP9" pad="2"/>
 <contactref element="JP7" pad="2"/>
-<wire x1="78.74" y1="35.56" x2="78.74" y2="38.1" width="0" layer="19" extent="1-1"/>
-<wire x1="73.66" y1="38.1" x2="78.74" y2="38.1" width="0" layer="19" extent="1-1"/>
-<wire x1="73.66" y1="35.56" x2="73.66" y2="38.1" width="0" layer="19" extent="1-1"/>
-<wire x1="68.58" y1="38.1" x2="73.66" y2="38.1" width="0" layer="19" extent="1-1"/>
-<wire x1="68.58" y1="33.02" x2="68.58" y2="38.1" width="0" layer="19" extent="1-1"/>
-<wire x1="60.96" y1="33.02" x2="68.58" y2="33.02" width="0" layer="19" extent="1-1"/>
-<wire x1="50.8" y1="22.86" x2="60.96" y2="33.02" width="0" layer="19" extent="1-1"/>
-<wire x1="48.26" y1="22.86" x2="50.8" y2="22.86" width="0" layer="19" extent="1-1"/>
-<wire x1="73.66" y1="20.32" x2="48.26" y2="22.86" width="0" layer="19" extent="1-1"/>
-<wire x1="73.66" y1="17.78" x2="73.66" y2="20.32" width="0" layer="19" extent="1-1"/>
-<wire x1="58.42" y1="20.32" x2="50.8" y2="22.86" width="0" layer="19" extent="1-1"/>
-<wire x1="58.42" y1="17.78" x2="58.42" y2="20.32" width="0" layer="19" extent="1-1"/>
-<wire x1="66.04" y1="20.32" x2="58.42" y2="20.32" width="0" layer="19" extent="1-1"/>
-<wire x1="66.04" y1="17.78" x2="66.04" y2="20.32" width="0" layer="19" extent="1-1"/>
-<wire x1="66.04" y1="50.8" x2="68.58" y2="38.1" width="0" layer="19" extent="1-1"/>
-<wire x1="66.04" y1="53.34" x2="66.04" y2="50.8" width="0" layer="19" extent="1-1"/>
+<wire x1="66.04" y1="50.8" x2="66.04" y2="53.34" width="0" layer="19" extent="1-1"/>
 <wire x1="55.88" y1="53.34" x2="66.04" y2="53.34" width="0" layer="19" extent="1-1"/>
 <wire x1="50.8" y1="53.34" x2="55.88" y2="53.34" width="0" layer="19" extent="1-1"/>
-<wire x1="43.18" y1="40.64" x2="50.8" y2="53.34" width="0" layer="19" extent="1-1"/>
+<wire x1="68.58" y1="40.64" x2="66.04" y2="50.8" width="0" layer="19" extent="1-1"/>
+<wire x1="73.66" y1="38.1" x2="68.58" y2="40.64" width="0" layer="19" extent="1-1"/>
+<wire x1="73.66" y1="35.56" x2="73.66" y2="38.1" width="0" layer="19" extent="1-1"/>
+<wire x1="78.74" y1="38.1" x2="73.66" y2="38.1" width="0" layer="19" extent="1-1"/>
+<wire x1="78.74" y1="35.56" x2="78.74" y2="38.1" width="0" layer="19" extent="1-1"/>
+<wire x1="68.58" y1="30.48" x2="73.66" y2="35.56" width="0" layer="19" extent="1-1"/>
+<wire x1="60.96" y1="33.02" x2="68.58" y2="30.48" width="0" layer="19" extent="1-1"/>
+<wire x1="66.04" y1="20.32" x2="68.58" y2="30.48" width="0" layer="19" extent="1-1"/>
+<wire x1="66.04" y1="17.78" x2="66.04" y2="20.32" width="0" layer="19" extent="1-1"/>
+<wire x1="73.66" y1="20.32" x2="66.04" y2="20.32" width="0" layer="19" extent="1-1"/>
+<wire x1="73.66" y1="17.78" x2="73.66" y2="20.32" width="0" layer="19" extent="1-1"/>
+<wire x1="58.42" y1="20.32" x2="66.04" y2="20.32" width="0" layer="19" extent="1-1"/>
+<wire x1="58.42" y1="17.78" x2="58.42" y2="20.32" width="0" layer="19" extent="1-1"/>
+<wire x1="50.8" y1="22.86" x2="58.42" y2="20.32" width="0" layer="19" extent="1-1"/>
+<wire x1="48.26" y1="22.86" x2="50.8" y2="22.86" width="0" layer="19" extent="1-1"/>
+<wire x1="38.1" y1="33.02" x2="48.26" y2="22.86" width="0" layer="19" extent="1-1"/>
+<wire x1="35.56" y1="30.48" x2="38.1" y2="33.02" width="0" layer="19" extent="1-1"/>
+<wire x1="43.18" y1="40.64" x2="38.1" y2="33.02" width="0" layer="19" extent="1-1"/>
 <wire x1="38.1" y1="43.18" x2="43.18" y2="40.64" width="0" layer="19" extent="1-1"/>
-<wire x1="38.1" y1="33.02" x2="43.18" y2="40.64" width="0" layer="19" extent="1-1"/>
-<wire x1="35.56" y1="30.48" x2="38.1" y2="33.02" width="0" layer="19" extent="1-1"/>
 <wire x1="25.4" y1="22.86" x2="35.56" y2="30.48" width="0" layer="19" extent="1-1"/>
 <wire x1="20.32" y1="43.18" x2="38.1" y2="43.18" width="0" layer="19" extent="1-1"/>
@@
 <contactref element="R1" pad="2"/>
 <contactref element="R2" pad="2"/>
+<wire x1="78.74" y1="33.02" x2="78.74" y2="50.8" width="0" layer="19" extent="1-1"/>
 <wire x1="73.66" y1="33.02" x2="78.74" y2="33.02" width="0" layer="19" extent="1-1"/>
-<wire x1="68.58" y1="30.48" x2="73.66" y2="33.02" width="0" layer="19" extent="1-1"/>
-<wire x1="58.42" y1="33.02" x2="68.58" y2="30.48" width="0" layer="19" extent="1-1"/>
+<wire x1="68.58" y1="33.02" x2="73.66" y2="33.02" width="0" layer="19" extent="1-1"/>
+<wire x1="58.42" y1="33.02" x2="68.58" y2="33.02" width="0" layer="19" extent="1-1"/>
 <wire x1="55.88" y1="33.02" x2="58.42" y2="33.02" width="0" layer="19" extent="1-1"/>
-<wire x1="78.74" y1="50.8" x2="78.74" y2="33.02" width="0" layer="19" extent="1-1"/>
 <wire x1="35.56" y1="33.02" x2="55.88" y2="33.02" width="0" layer="19" extent="1-1"/>
 <wire x1="33.02" y1="33.02" x2="35.56" y2="33.02" width="0" layer="19" extent="1-1"/>
@@
 <contactref element="T2" pad="E"/>
 <wire x1="73.66" y1="40.64" x2="78.74" y2="40.64" width="0" layer="19" extent="1-1"/>
-<wire x1="68.58" y1="40.64" x2="73.66" y2="40.64" width="0" layer="19" extent="1-1"/>
 <wire x1="71.12" y1="45.72" x2="73.66" y2="40.64" width="0" layer="19" extent="1-1"/>
-<wire x1="48.26" y1="40.64" x2="68.58" y2="40.64" width="0" layer="19" extent="1-1"/>
+<wire x1="68.58" y1="38.1" x2="73.66" y2="40.64" width="0" layer="19" extent="1-1"/>
+<wire x1="48.26" y1="40.64" x2="68.58" y2="38.1" width="0" layer="19" extent="1-1"/>
 <wire x1="45.72" y1="40.64" x2="48.26" y2="40.64" width="0" layer="19" extent="1-1"/>
 <wire x1="25.4" y1="40.64" x2="45.72" y2="40.64" width="0" layer="19" extent="1-1"/>
@@
 <contactref element="LED1" pad="A"/>
 <contactref element="R1" pad="1"/>
-<wire x1="71.12" y1="50.8" x2="71.12" y2="48.26" width="0" layer="19" extent="1-1"/>
+<wire x1="71.12" y1="48.26" x2="71.12" y2="50.8" width="0" layer="19" extent="1-1"/>
 </signal>
 <signal name="N$1">
@@
 <wire x1="17.78" y1="50.8" x2="22.86" y2="48.26" width="0" layer="19" extent="1-1"/>
 <wire x1="15.24" y1="45.72" x2="17.78" y2="50.8" width="0" layer="19" extent="1-1"/>
-<wire x1="17.78" y1="40.64" x2="17.78" y2="50.8" width="0" layer="19" extent="1-1"/>
+<wire x1="17.78" y1="40.64" x2="15.24" y2="45.72" width="0" layer="19" extent="1-1"/>
 </signal>
 <signal name="N$3">

Commit message: Update eagle files
Parts:
- JP1, JP2: device pinhead:1X04 -> pinhead:1X03
- moved R1 7.18 mm to (80.0, 45.7)
- moved R11 7.18 mm to (55.9, 49.5)
- moved R16 7.18 mm to (58.4, 49.5)
- moved R2 5.08 mm to (12.7, 36.8)
- moved LED1 3.59 mm to (73.7, 44.5)
- moved R15 2.54 mm to (63.5, 24.1)
- moved JP7 2.54 mm to (64.8, 15.2)
- moved JP9 2.54 mm to (57.1, 15.2)
- moved T1 2.54 mm to (12.7, 50.8)
- moved T2 2.54 mm to (12.7, 45.7)
- moved C3 2.54 mm to (22.9, 48.3)
- moved C4 2.54 mm to (17.8, 27.9)
- moved C5 2.54 mm to (48.3, 49.5)
- moved C6 2.54 mm to (43.2, 30.5)
- moved C7 2.54 mm to (34.3, 33.0)
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Connections:
- net GND: no longer JP1.3, JP2.3
- net V-: now also JP1.3, JP2.3; no longer JP1.4, JP2.4
Routing:
- net GND: track 0.00 -> 316.8 mm, vias 0 -> 6
- net V+: track 0.00 -> 101.2 mm
- net V-: track 0.00 -> 81.3 mm
- net N$10: track 0.00 -> 77.3 mm, vias 0 -> 6
- net N$7: track 0.00 -> 63.5 mm, vias 0 -> 2
- net N$2: track 0.00 -> 17.8 mm
- net N$6: track 0.00 -> 13.8 mm
- net N$14: track 0.00 -> 11.2 mm
- net N$9: track 0.00 -> 7.62 mm
- net N$12: track 0.00 -> 7.62 mm
- net N$8: track 0.00 -> 7.62 mm
- net N$17: track 0.00 -> 7.62 mm
- net N$21: track 0.00 -> 7.62 mm
- net N$3: track 0.00 -> 7.62 mm
- net N$11: track 0.00 -> 7.62 mm
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